File: schematics/all/power_supply_unit.sch (EAGLE design)
At the start: 0 parts

Commit message: added power supply schematics etc
Parts:
- added G1: BATTERY_12V_8XAA, martins-parts:BATTERY_12V_8XAA
- added R1: 10k 1%, resistor:R-EU_0207/10
- added R2: 4.7k 1%, resistor:R-EU_0207/10
- added U$1, U$2: STEP_DOWN_CONVERTER, martins-parts:STEP_DOWN_CONVERTER
- added U$3: ACS71X_CURRENT_SENSOR, martins-parts:ACS71X_CURRENT_SENSOR
Connections:
- new net +5V: U$3.VCC
- new net GND: G1.-, R2.1, U$3.GND
- new net I_BATT_SENSE: U$3.VOUT
- new net N$1: G1.+, R1.2, U$3.IP-
- new net N$2: U$3.IP+
- new net U_BATT_SENSE: R1.1, R2.2
Other:
- note added: "(C) 2016 by Martin Hepp, DO1MFH martin.hepp@unibw.de"
- note added: "Power Supply Unit for High Altitude Balloon Project"
- note added: "To ADS1015 12-Bit ADC - 4 Channel with Programmable Gain Amplifier Module"
- note added: "To DORJI DRA818V Transceiver Module"
- note added: "To Raspberry Pi 1, 2, and 3"
Changed lines of the file:
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@@
 <?xml version="1.0" encoding="utf-8"?>
 <!DOCTYPE eagle SYSTEM "eagle.dtd">
-<eagle version="7.5.0">
+<eagle version="7.6.0">
 <drawing>
 <settings>
@@
 <setting verticaltext="up"/>
 </settings>
-<grid distance="0.1" unitdist="inch" unit="inch" style="lines" multiple="1" display="no" altdistance="0.01" altunitdist="inch" altunit="inch"/>
+<grid distance="0.1" unitdist="inch" unit="inch" style="lines" multiple="1" display="yes" altdistance="0.01" altunitdist="inch" altunit="inch"/>
 <layers>
 <layer number="1" name="Top" color="4" fill="1" visible="no" active="no"/>
@@
 <layer number="97" name="Info" color="7" fill="1" visible="yes" active="yes"/>
 <layer number="98" name="Guide" color="6" fill="1" visible="yes" active="yes"/>
+<layer number="99" name="SpiceOrder" color="5" fill="1" visible="yes" active="yes"/>
+<layer number="100" name="Parts" color="7" fill="1" visible="yes" active="yes"/>
+<layer number="250" name="Descript" color="7" fill="1" visible="yes" active="yes"/>
+<layer number="251" name="SMDround" color="7" fill="1" visible="yes" active="yes"/>
 </layers>
 <schematic xreflabel="%F%N/%S.%C%R" xrefpart="/%S.%C%R">
@@
 <parts>
 <part name="FRAME1" library="frames" deviceset="DINA4_L" device=""/>
+<part name="G1" library="martins-parts" deviceset="BATTERY_12V_8XAA" device=""/>
+<part name="R1" library="resistor" deviceset="R-EU_" device="0207/10" value="10k 1%"/>
+<part name="R2" library="resistor" deviceset="R-EU_" device="0207/10" value="4.7k 1%"/>
+<part name="GND1" library="supply1" deviceset="GND" device=""/>
+<part name="GND5" library="supply1" deviceset="GND" device=""/>
+<part name="U$3" library="martins-parts" deviceset="ACS71X_CURRENT_SENSOR" device=""/>
+<part name="U$1" library="martins-parts" deviceset="STEP_DOWN_CONVERTER" device=""/>
+<part name="U$2" library="martins-parts" deviceset="STEP_DOWN_CONVERTER" device=""/>
+<part name="GND2" library="supply1" deviceset="GND" device=""/>
+<part name="GND3" library="supply1" deviceset="GND" device=""/>
+<part name="GND4" library="supply1" deviceset="GND" device=""/>
+<part name="GND6" library="supply1" deviceset="GND" device=""/>
+<part name="GND7" library="supply1" deviceset="GND" device=""/>
+<part name="GND8" library="supply1" deviceset="GND" device=""/>
+<part name="GND9" library="supply1" deviceset="GND" device=""/>
+<part name="P+1" library="supply1" deviceset="+5V" device=""/>
 </parts>
 <sheets>
 <sheet>
 <plain>
+<text x="187.96" y="134.62" size="2.54" layer="97">To Raspberry Pi 1, 2, and 3</text>
+<text x="187.96" y="99.06" size="2.54" layer="97">To DORJI DRA818V Transceiver Module</text>
+<text x="187.96" y="60.96" size="2.54" layer="97">To ADS1015 12-Bit ADC - 4 Channel
+with Programmable Gain Amplifier Module</text>
+<text x="132.08" y="165.1" size="6.4516" layer="94" align="center">Power Supply Unit for
+High Altitude Balloon Project</text>
+<text x="5.08" y="7.62" size="1.778" layer="94">(C) 2016 by Martin Hepp, DO1MFH
+martin.hepp@unibw.de</text>
 </plain>
 <instances>
 <instance part="FRAME1" gate="G$1" x="0" y="0"/>
 <instance part="FRAME1" gate="G$2" x="162.56" y="0"/>
+<instance part="G1" gate="G$1" x="15.24" y="104.14" rot="R90"/>
+<instance part="R1" gate="G$1" x="27.94" y="96.52" rot="R90"/>
+<instance part="R2" gate="G$1" x="27.94" y="86.36" rot="R90"/>
+<instance part="GND1" gate="1" x="15.24" y="78.74"/>
+<instance part="GND5" gate="1" x="27.94" y="78.74"/>
+<instance part="U$3" gate="G$1" x="53.34" y="119.38"/>
+<instance part="U$1" gate="G$1" x="116.84" y="142.24"/>
+<instance part="U$2" gate="G$1" x="116.84" y="106.68"/>
+<instance part="GND2" gate="1" x="109.22" y="83.82"/>
+<instance part="GND3" gate="1" x="109.22" y="119.38"/>
+<instance part="GND4" gate="1" x="149.86" y="119.38"/>
+<instance part="GND6" gate="1" x="149.86" y="83.82"/>
+<instance part="GND7" gate="1" x="170.18" y="83.82"/>
+<instance part="GND8" gate="1" x="170.18" y="119.38"/>
+<instance part="GND9" gate="1" x="68.58" y="104.14"/>
+<instance part="P+1" gate="1" x="53.34" y="142.24"/>
 </instances>
 <busses>
 </busses>
 <nets>
+<net name="U_BATT_SENSE" class="0">
+<segment>
+<pinref part="R1" gate="G$1" pin="1"/>
+<pinref part="R2" gate="G$1" pin="2"/>
+<wire x1="27.94" y1="91.44" x2="55.88" y2="91.44" width="0.1524" layer="91"/>
+<junction x="27.94" y="91.44"/>
+<label x="164.084" y="59.436" size="1.778" layer="95"/>
+<wire x1="55.88" y1="91.44" x2="55.88" y2="58.42" width="0.1524" layer="91"/>
+<wire x1="55.88" y1="58.42" x2="182.88" y2="58.42" width="0.1524" layer="91"/>
+</segment>
+</net>
+<net name="GND" class="0">
+<segment>
+<pinref part="R2" gate="G$1" pin="1"/>
+<pinref part="GND5" gate="1" pin="GND"/>
+</segment>
+<segment>
+<pinref part="GND3" gate="1" pin="GND"/>
+<wire x1="109.22" y1="121.92" x2="109.22" y2="129.54" width="0.1524" layer="91"/>
+</segment>
+<segment>
+<pinref part="GND4" gate="1" pin="GND"/>
+<wire x1="149.86" y1="129.54" x2="149.86" y2="121.92" width="0.1524" layer="91"/>
+</segment>
+<segment>
+<pinref part="GND6" gate="1" pin="GND"/>
+<wire x1="149.86" y1="93.98" x2="149.86" y2="86.36" width="0.1524" layer="91"/>
+</segment>
+<segment>
+<pinref part="GND2" gate="1" pin="GND"/>
+<wire x1="109.22" y1="93.98" x2="109.22" y2="86.36" width="0.1524" layer="91"/>
+</segment>
+<segment>
+<wire x1="182.88" y1="93.98" x2="170.18" y2="93.98" width="0.1524" layer="91"/>
+<wire x1="170.18" y1="93.98" x2="170.18" y2="86.36" width="0.1524" layer="91"/>
+<pinref part="GND7" gate="1" pin="GND"/>
+<label x="177.292" y="94.742" size="1.778" layer="95"/>
+</segment>
+<segment>
+<pinref part="GND8" gate="1" pin="GND"/>
+<wire x1="170.18" y1="121.92" x2="170.18" y2="129.54" width="0.1524" layer="91"/>
+<wire x1="170.18" y1="129.54" x2="182.88" y2="129.54" width="0.1524" layer="91"/>
+<label x="177.292" y="130.302" size="1.778" layer="95"/>
+</segment>
+<segment>
+<pinref part="GND1" gate="1" pin="GND"/>
+<pinref part="G1" gate="G$1" pin="-"/>
+<wire x1="15.24" y1="81.28" x2="15.24" y2="83.82" width="0.1524" layer="91"/>
+</segment>
+<segment>
+<pinref part="GND9" gate="1" pin="GND"/>
+<pinref part="U$3" gate="G$1" pin="GND"/>
+<wire x1="68.58" y1="106.68" x2="68.58" y2="111.76" width="0.1524" layer="91"/>
+</segment>
+</net>
+<net name="N$1" class="0">
+<segment>
+<pinref part="G1" gate="G$1" pin="+"/>
+<wire x1="15.24" y1="111.76" x2="15.24" y2="119.38" width="0.1524" layer="91"/>
+<pinref part="R1" gate="G$1" pin="2"/>
+<wire x1="15.24" y1="119.38" x2="27.94" y2="119.38" width="0.1524" layer="91"/>
+<wire x1="27.94" y1="119.38" x2="27.94" y2="101.6" width="0.1524" layer="91"/>
+<pinref part="U$3" gate="G$1" pin="IP-"/>
+<wire x1="38.1" y1="111.76" x2="33.02" y2="111.76" width="0.1524" layer="91"/>
+<wire x1="33.02" y1="111.76" x2="33.02" y2="119.38" width="0.1524" layer="91"/>
+<wire x1="33.02" y1="119.38" x2="27.94" y2="119.38" width="0.1524" layer="91"/>
+<junction x="27.94" y="119.38"/>
+</segment>
+</net>
+<net name="N$2" class="0">
+<segment>
+<pinref part="U$3" gate="G$1" pin="IP+"/>
+<wire x1="38.1" y1="127" x2="38.1" y2="147.32" width="0.1524" layer="91"/>
+<wire x1="38.1" y1="147.32" x2="104.14" y2="147.32" width="0.1524" layer="91"/>
+<wire x1="104.14" y1="147.32" x2="104.14" y2="139.7" width="0.1524" layer="91"/>
+<wire x1="104.14" y1="139.7" x2="104.14" y2="104.14" width="0.1524" layer="91"/>
+<wire x1="104.14" y1="104.14" x2="109.22" y2="104.14" width="0.1524" layer="91"/>
+<wire x1="109.22" y1="139.7" x2="104.14" y2="139.7" width="0.1524" layer="91"/>
+<junction x="104.14" y="139.7"/>
+</segment>
+</net>
+<net name="+5.2V" class="0">
+<segment>
+<wire x1="149.86" y1="139.7" x2="182.88" y2="139.7" width="0.1524" layer="91"/>
+<label x="176.53" y="140.208" size="1.778" layer="95"/>
+</segment>
+</net>
+<net name="+4.2V" class="0">
+<segment>
+<wire x1="149.86" y1="104.14" x2="182.88" y2="104.14" width="0.1524" layer="91"/>
+<label x="176.53" y="104.902" size="1.778" layer="95"/>
+</segment>
+</net>
+<net name="I_BATT_SENSE" class="0">
+<segment>
+<pinref part="U$3" gate="G$1" pin="VOUT"/>
+<wire x1="68.58" y1="127" x2="81.28" y2="127" width="0.1524" layer="91"/>
+<label x="165.608" y="69.596" size="1.778" layer="95"/>
+<wire x1="81.28" y1="127" x2="81.28" y2="68.58" width="0.1524" layer="91"/>
+<wire x1="81.28" y1="68.58" x2="182.88" y2="68.58" width="0.1524" layer="91"/>
+</segment>
+</net>
+<net name="+5V" class="0">
+<segment>
+<pinref part="U$3" gate="G$1" pin="VCC"/>
+<pinref part="P+1" gate="1" pin="+5V"/>
+<wire x1="53.34" y1="137.16" x2="53.34" y2="139.7" width="0.1524" layer="91"/>
+</segment>
+</net>
 </nets>
 </sheet>
@@
 </schematic>
 </drawing>
+<compatibility>
+<note version="6.3" minversion="6.2.2" severity="warning">
+Since Version 6.2.2 text objects can contain more than one line,
+which will not be processed correctly with this version.
+</note>
+</compatibility>
 </eagle>
