File: schematics/all/overview.sch (EAGLE design)
At the start: 0 parts

Commit message: next version
Parts:
- added BATT_TEMPERATURE: DS1820TO92-BATT, Ava:DS1820TO92
- added R1: 4.7k, resistor:R-EU_0207/7
- added U$1: LPF_160MHZ, martins-parts:LPF_160MHZ
- added U$2: RASPBERRY-PI+HEADERONLY, Ava:RASPBERRY-PI+HEADERONLY
- added U$4, U$5: DS1820TO92, Ava:DS1820TO92
- added U1: DRA818, dorji_module:DRA818
Connections:
- new net +4.2V: U1.VBAT
- new net GND: BATT_TEMPERATURE.GND, U$1.RF_GND@1, U$4.GND, U$5.GND, U1.GND$1, U1.GND$2, U1.GND$3, U1.GND$4, U1.GND$5
- new net N$1: U$1.RF_IN, U1.ANT
- new net N$2: U1.RXD
- new net N$3: U1.TXD
- new net N$4: BATT_TEMPERATURE.DQ, R1.2, U$4.DQ, U$5.DQ
- new net N$5: BATT_TEMPERATURE.VCC, R1.1, U$4.VCC, U$5.VCC
Other:
- note added: "Battery Temperature"
- note added: "Outside Temperature"
